Commit message: le bot is viewable

File: description/robot_core.xacro (robot description, xacro)
@@ -1,4 +1,5 @@
 <?xml version="1.0"?>
-<robot xmlns:xacro="http://www.ros.org/wiki/xacro"  >
+<robot xmlns:xacro="http://www.ros.org/wiki/xacro">
+    <xacro:include filename="inertial_macro.xacro"/>
     <material name="white">
         <color rgba="1 1 1 1" />
@@ -28,6 +29,15 @@
                 <box size="0.3 0.24 0.122" />
             </geometry>
-            <meterial name="white"/>
+            <material name="white"/>
         </visual>
+        <collision>
+            <origin xyz="0.15 0 0.061"/>
+            <geometry>
+                <box size="0.3 0.24 0.122" />
+            </geometry>
+        </collision>
+        <xacro:inertial_box mass="0.5" x="0.3" y="0.24" z="0.122">
+            <origin xyz="0.15 0 0.061" rpy="0 0 0"/>
+        </xacro:inertial_box>
     </link>
     <!--  LEFT WHEEL LINK  -->
@@ -45,4 +55,12 @@
             <material name="blue"/>
         </visual>
+        <collision>
+            <geometry>
+                <cylinder radius="0.05" length="0.04"/>
+            </geometry>
+        </collision>
+        <xacro:inertial_cylinder mass="0.1" length="0.04" radius="0.05">
+            <origin xyz="0 0 0" rpy="0 0 0"/>
+        </xacro:inertial_cylinder>
     </link>
     <!--  RIGHT WHEEL LINK  -->
@@ -60,4 +78,34 @@
             <material name="blue"/>
         </visual>
+        <collision>
+            <geometry>
+                <cylinder radius="0.05" length="0.04"/>
+            </geometry>
+        </collision>
+        <xacro:inertial_cylinder mass="0.1" length="0.04" radius="0.05">
+            <origin xyz="0 0 0" rpy="0 0 0"/>
+        </xacro:inertial_cylinder>
+    </link>
+    <!--  CASTER WHEEL LINK  -->
+    <joint name="caster_wheel_joint" type="fixed">
+        <parent link="chassis"/>
+        <child link="caster_wheel"/>
+        <origin xyz="0.24 0 0"/>
+    </joint>
+    <link name="caster_wheel">
+        <visual>
+            <geometry>
+                <sphere radius="0.05"/>
+            </geometry>
+            <material name="black"/>
+        </visual>
+        <collision>
+            <geometry>
+                <sphere radius="0.05"/>
+            </geometry>
+        </collision>
+        <xacro:inertial_sphere mass="0.01" radius="0.05">
+            <origin xyz="0 0 0" rpy="0 0 0"/>
+        </xacro:inertial_sphere>
     </link>
 </robot>

Commit message: idk

File: description/robot_core.xacro (robot description, xacro)
@@ -16,4 +16,12 @@
     <!--  BASE LINK  -->
     <link name="base_link">
+    </link>
+    <!--  BASE FOOTPRINT LINK  -->
+    <joint name="base_footprint_joint" type="fixed">
+        <parent link="base_link"/>
+        <child link="base_footprint"/>
+        <origin xyz="0 0 0" rpy="0 0 0"/>
+    </joint>
+    <link name="base_footprint">
     </link>
     <!--  CHASSIS LINK  -->
